Commit message: Add the FT 300 and the Wrist Camera to the wrist stack
The real robot is UR5e -> FT 300 -> Wrist Camera -> 2F-85; the model had
only the gripper, so the planner thought the tool started 55 mm closer to
the flange than it does. The D435i bracket stays where it was.

  tool0 -> ft300_coupling -> ft300_sensor -> wrist_camera -> 2F-85 -> D435i
           z=0              z=41.5 mm       z=48.3 mm       z=55.0 mm

FT 300 meshes are the official ros-industrial ones (BSD, LICENSE kept
beside them), measured rather than trusted: coupling plate 75.0 x 74.9 x
13.0 mm, sensor body 75.0 x 75.0 x 34.8 mm, and the official mounting
transform seats them so the assembly adds 41.5 mm.

Robotiq publishes NO URDF or mesh for the Wrist Camera - the ROS wiki says
it is unsupported, and the one third-party repo that references a mesh for
it contains no mesh files at all. It is therefore a box at the documented
outer dimensions, 87.5 x 75 x 22.4 mm, adding 13.5 mm with a 2-finger
gripper. Geometry only: no optical frame, not in CAMERAS. The camera that
actually maps is still the D435i.

Orientation was read off the hardware photos - the camera's two LEDs and
lens sit in a row along its long edge, parallel to the direction the
fingers open - and confirmed by the owner against the real assembly, along
with the stack height.

Two things this turned up.

Isaac Sim's URDF importer does not sanitise mesh FILENAMES into USD prim
names. The coupling plate ships as robotiq_ft300-G-062-COUPLING_G-50-4M6-
1D6_20181119.STL, and a hyphen is illegal in a prim name, so it produced a
null prim and the ENTIRE import failed with "RuntimeError: Used null prim"
- naming no file. It does sanitise link and joint names and logs that it
did, which is what makes the omission easy to miss. Isolated by bisection:
boxing that one mesh imports fine, renaming it imports fine, converting it
to .obj does not. Stored as ft300_coupling.STL. HANDOVER section 4.

Collision sphere centres are in the LINK's own frame, and I wrote the
first set in tool0's. The camera's spheres floated 48 mm up inside the
gripper - invisible, useless, and silent - which the owner spotted in the
viewer. ft300_sensor is additionally flipped 180 deg about Y by its
mounting transform, so all twelve FT 300 spheres now live on
ft300_coupling, the one link in the stack whose joint is identity relative
to tool0; ft300_sensor keeps its mesh and carries none. Verified by
forward kinematics that every link's spheres now span its own geometry.

check_robot_cfg.py was broken for this robot and had been: it did not trim
tool_frames, so plan_pose demanded a goal for camera_link too. Fixed the
same way planner_server.build() does it, so the documented verification
step runs again.

Verified: 81 spheres, plan_pose success in 24 ms, URDF imports clean, and
a full demo run gave 89 detour plans with 0 self-hits at the end. A new
startup transient is recorded in HANDOVER section 8 - 35 early plans fail
on a self-mapped fingertip before frustum decay clears it, then it
recovers. self_mask_margin was tuned for the shorter tool and wants its
own A/B.

Co-Authored-By: Claude Opus 5 <noreply@anthropic.com>

File: assets/robot/ur_description/ur5e_robotiq_2f_85.urdf (robot description, URDF)
Before this commit: robot ur5e_robotiq_2f_85, 25 links, 24 joints
Links:
- added link ft300_coupling; collision mesh filename=../robotiq/ft300/meshes/collision/ft300_coupling.STL; visual mesh filename=../robotiq/ft300/meshes/visual/ft300_coupling.STL
- added link ft300_sensor; collision mesh filename=../robotiq/ft300/meshes/collision/robotiq_ft300.STL; visual mesh filename=../robotiq/ft300/meshes/visual/robotiq_ft300.STL
- added link wrist_camera; collision box size=0.0875 0.0750 0.0224; visual box size=0.0875 0.0750 0.0224
Joints:
- added joint ft300_coupling_joint: type fixed, parent tool0, child ft300_coupling, origin xyz=0 0 0 rpy=0 0 0
- added joint ft300_sensor_joint: type fixed, parent ft300_coupling, child ft300_sensor, origin xyz=0 0 0.0415 rpy=0 3.14159265 0
- added joint wrist_camera_joint: type fixed, parent tool0, child wrist_camera, origin xyz=0 0 0.0483 rpy=0 0 0.0000
- joint gripper_base_joint: origin xyz=0.0 0.0 0.0 rpy=0.0 0.0 1.57 -> xyz=0.0 0.0 0.0550 rpy=0.0 0.0 1.57

Commit message: Actuate the 2F-85: one driving joint, five mimics, locked out of the cspace
The fingers were rigid collision geometry. They now move, while the planner
still solves the same six arm joints.

The 4-bar linkage needs a loop closure URDF cannot express, so this takes
the approximation every Robotiq ROS package takes: left_outer_knuckle_joint
drives (0 rad open, 0.8 closed) and five <mimic> joints follow. cuRobo
0.7.7's Kinova model, which these links came from, made them all fixed but
kept origins identical to ros-industrial's macro - checked joint by joint -
so restoring the articulation moves nothing at angle 0.

The config locks the driving joint at 0.0 (franka.yml is the precedent).
Locking is not fixing: cuRobo still places the fingers and their spheres, so
it knows the gripper's shape. Measured over the stroke, a finger sphere
moves 48.5 mm while every arm sphere moves 0.000 mm, and the cspace stays
six joints. Locked OPEN on purpose - the widest the gripper gets, so a route
that clears open stays clear while it closes; the reverse does not hold.

Three things this turned up.

The returned trajectory is WIDER than the cspace: a 6-DOF plan comes back 7
columns with the locked joint appended, and only interpolated_trajectory.
joint_names says so. handle_plan now selects columns by name. Trusting the
width would have handed the client a vector one longer than the joint list
it was given, with nothing to say so - the arm mapping would just be off by
one.

The demo's joint mapping had to go. curobo_names.index(j) over every sim
joint raises the moment the simulator has a joint the planner has not heard
of, which is now. Arm and gripper are addressed by joint_indices instead, so
an arm command cannot disturb the fingers.

Stroke timing has to come from the velocity limit, not a guess. The joints
cap at 2.0 rad/s, so 0.8 rad needs 24 steps at 60 Hz; ten-step ramps left
the gripper stranded at +0.334 rad when the next plan began. Sized from the
limit it returns to +0.001..+0.017 rad every cycle.

Isaac Sim imports <mimic> natively, so only the driving joint is commanded.

Regression, both cameras: 55 plans, 0 failures, all on detour routes, 0
self-hits in all 358 map reports, and the gripper cycling correctly at every
target. Tracking error 0.09-0.73 deg, up from 0.08-0.27 - the gripper's
reaction disturbs the arm slightly, recorded in section 10 rather than
smoothed over.

Geometric actuation only: DRAG_CUBE is a VisualCuboid with no physics, so
there is still nothing to grasp.

Co-Authored-By: Claude Opus 5 <noreply@anthropic.com>

File: assets/robot/ur_description/ur5e_robotiq_2f_85.urdf (robot description, URDF)
Before this commit: robot ur5e_robotiq_2f_85, 28 links, 27 joints
Joints:
- joint left_inner_finger_joint: axis (none) -> 1 0 0; limit (none) -> lower=0 upper=0.8757 effort=1000 velocity=2.0; mimic (none) -> joint=left_outer_knuckle_joint multiplier=-1.0 offset=0; type fixed -> revolute
- joint left_inner_knuckle_joint: axis (none) -> 1 0 0; limit (none) -> lower=0 upper=0.8757 effort=1000 velocity=2.0; mimic (none) -> joint=left_outer_knuckle_joint multiplier=1.0 offset=0; type fixed -> revolute
- joint left_outer_knuckle_joint: axis (none) -> 1 0 0; limit (none) -> lower=0 upper=0.8 effort=1000 velocity=2.0; type fixed -> revolute
- joint right_inner_finger_joint: axis (none) -> 1 0 0; limit (none) -> lower=0 upper=0.8757 effort=1000 velocity=2.0; mimic (none) -> joint=left_outer_knuckle_joint multiplier=-1.0 offset=0; type fixed -> revolute
- joint right_inner_knuckle_joint: axis (none) -> 1 0 0; limit (none) -> lower=0 upper=0.8757 effort=1000 velocity=2.0; mimic (none) -> joint=left_outer_knuckle_joint multiplier=1.0 offset=0; type fixed -> revolute
- joint right_outer_knuckle_joint: axis (none) -> 1 0 0; limit (none) -> lower=0 upper=0.81 effort=1000 velocity=2.0; mimic (none) -> joint=left_outer_knuckle_joint multiplier=1.0 offset=0; type fixed -> revolute

Commit message: Drop <mimic> from the URDF: PhysX rejects it and breaks the articulation
The gripper came apart on screen. Reported from a screenshot, not from any
number the project was printing.

PhysX refuses to build a mimic constraint - "the revolute joint at ...
needs a finite limit set to be used by the mimic joint feature", though
every one of them has lower="0" upper="0.8757" - and the failure is not
contained. It takes the whole articulation with it. Stripping the tags
takes the error count 1 -> 0 and the articulation builds.

The coupling moves to rig.ROBOTS[...]["gripper_joints"], joint to
multiplier, and three consumers derive from it: the URDF builder takes the
SIGN of each joint's limits, the config builder locks all six, the
simulator commands all six. One place to change.

Signed limits were the second half of it. A joint with multiplier -1
travels negative, so lower="0" pins it at zero - driven explicitly, the
four positive joints tracked a close command perfectly while both
inner_finger joints sat at -0.000. Upstream has the same lower="0" with
multiplier="-1" and gets away with it only because a mimic constraint
computes the follower instead of commanding it through its own limit.

What let this through: I verified the gripper by measuring cuRobo's
collision spheres, which moved correctly. cuRobo resolves the coupling
itself and never touches PhysX, so it reported a perfect gripper while the
simulator's was in pieces. Same URDF, two entirely separate paths.
Checking the planner is not checking the simulator, and the importer
logging that it saw the <mimic> tags is not the physics engine agreeing to
enforce them. Both sides are now measured.

Verified. PhysX: all six joints track a commanded stroke to within 0.3
mrad, inner_finger reaching -0.800 where it previously sat at -0.000, zero
mimic errors. cuRobo: spheres move 47.0 mm open to closed, every arm
sphere 0.000 mm, cspace still six joints. Regression: 55 plans, 0
failures, all detours, 0 self-hits across 359 map reports, gripper
returning to +0.003..+0.004 rad each cycle.

Tracking error is back to 0.09-0.19 deg from 0.09-0.73. That 0.73 was the
broken linkage tearing at the arm in PhysX, and I had recorded it in
section 10 as the gripper's reaction force. Corrected.

The trajectory is now 12 columns wide rather than 7 - six locked joints
appended instead of one. handle_plan already selected columns by name, so
nothing broke; anything hard-coded to the old width would have.

Co-Authored-By: Claude Opus 5 <noreply@anthropic.com>

File: assets/robot/ur_description/ur5e_robotiq_2f_85.urdf (robot description, URDF)
Before this commit: robot ur5e_robotiq_2f_85, 28 links, 27 joints
Joints:
- joint left_inner_finger_joint: limit lower=0 upper=0.8757 effort=1000 velocity=2.0 -> lower=-0.8757 upper=0.0 effort=1000 velocity=2.0; mimic joint=left_outer_knuckle_joint multiplier=-1.0 offset=0 -> (none)
- joint left_inner_knuckle_joint: limit lower=0 upper=0.8757 effort=1000 velocity=2.0 -> lower=0.0 upper=0.8757 effort=1000 velocity=2.0; mimic joint=left_outer_knuckle_joint multiplier=1.0 offset=0 -> (none)
- joint left_outer_knuckle_joint: limit lower=0 upper=0.8 effort=1000 velocity=2.0 -> lower=0.0 upper=0.8 effort=1000 velocity=2.0
- joint right_inner_finger_joint: limit lower=0 upper=0.8757 effort=1000 velocity=2.0 -> lower=-0.8757 upper=0.0 effort=1000 velocity=2.0; mimic joint=left_outer_knuckle_joint multiplier=-1.0 offset=0 -> (none)
- joint right_inner_knuckle_joint: limit lower=0 upper=0.8757 effort=1000 velocity=2.0 -> lower=0.0 upper=0.8757 effort=1000 velocity=2.0; mimic joint=left_outer_knuckle_joint multiplier=1.0 offset=0 -> (none)
- joint right_outer_knuckle_joint: limit lower=0 upper=0.81 effort=1000 velocity=2.0 -> lower=0.0 upper=0.81 effort=1000 velocity=2.0; mimic joint=left_outer_knuckle_joint multiplier=1.0 offset=0 -> (none)
