Commit message: Get the UR5 running in Isaac Sim: four separate faults
The demo did not run after the model swap. Four independent things were
wrong, each measured before it was touched.

1. wrist_1 would not hold still -- 770 mrad of drift at HOME while every
   other joint stayed inside 5 mrad, and it read as a loose joint on screen.
   This description has 26 links that are pure coordinate frames with no mass
   and no geometry, and the importer gives each of them "a small isotropic
   inertia"; twenty of those hanging off the wrist wreck the articulation
   solver. Merging the fixed joints drops it to 4.4 mrad. The 4-bar pin was
   ruled out first: 663 mrad with it removed.

   Merging discards the frames' prims, so camera_link no longer exists to
   hang the D435i on. frame_prim() walks the URDF to the nearest link that
   does have a prim and puts an Xform back, which costs PhysX nothing.

2. Every plan failed. The eight base_link_inertia spheres added in the last
   commit sit inside the table cuboid for every configuration -- 17.1 mm of
   penetration, at HOME and at both goals -- so the planner called the robot
   in collision whatever it was asked. cuRobo's ur5e.yml leaves the base bare
   and that is not an oversight: nothing the planner does moves the base.

3. The goals were still refused, by the mapped table rather than the real
   one. A UR5 (CB3) shoulder sits at z = 89 mm, 73 mm lower than the
   e-Series arm cuRobo's config was tuned on, so the upper arm's spheres are
   permanently inside the map's inflated copy of a surface the planner
   already knows exactly. Depth below floor_z is no longer fused; the real
   table is still in the static scene and still checked. The map goes from
   16 000 voxels to the 300 that are the obstacle.

   Sphere protrusion was tightened on the way: shoulder_link and
   upper_arm_link now clamp to their own geometry instead of hanging 14-20 mm
   below the metal.

4. With that fixed the plans succeeded at 440 ms, because the demo had been
   run with --no-cuda-graph to get this far. With graphs on, everything
   failed from the first call. Building the approach IK from the planner's
   own ik_solver_config corrupts the planner:

       second solver from the shared config : plan FAIL, FAIL, FAIL
       second solver from a deep copy       : plan ok,   ok,   ok
       no second solver at all              : plan ok,   ok,   ok

   Reproduced on cuRobo's shipped ur5e config too, so it is not this robot.
   A deep copy fixes it and the two solvers still behave differently, which
   is the point of having both: a pose buried in the table is refused by the
   collision-aware one and solved by the free one. Plans are back to 50 ms.

Also folded in: the joint-limit clip to +/-180 deg, which used to be a
separate tool run by hand between the two builders and was lost in the swap;
and the failure diagnostics that found (2) and (3) -- the planner now reports
clearance to the map rather than only "nothing inside the robot", and says
whether a failed plan's GOAL is reachable, solving it without collisions if
it has to just to have something to measure.

demo_cube runs: 81 waypoints, 51 ms a plan, the arm shuttling between targets.
baseline and pick_place are not re-checked yet, and README and HANDOVER still
describe the old robot.

Co-Authored-By: Claude Opus 5 <noreply@anthropic.com>

File: assets/robot/ur5_robotiq/ur5_robotiq.urdf (robot description, URDF)
Before this commit: robot ur5_robotiq, 46 links, 45 joints
Joints:
- joint shoulder_lift_joint: limit lower=-6.283185307179586 upper=6.283185307179586 effort=150.0 velocity=3.141592653589793 -> lower=-3.141593 upper=3.141593 effort=150.0 velocity=3.141592653589793
- joint shoulder_pan_joint: limit lower=-6.283185307179586 upper=6.283185307179586 effort=150.0 velocity=3.141592653589793 -> lower=-3.141593 upper=3.141593 effort=150.0 velocity=3.141592653589793
- joint wrist_1_joint: limit lower=-6.283185307179586 upper=6.283185307179586 effort=28.0 velocity=3.141592653589793 -> lower=-3.141593 upper=3.141593 effort=28.0 velocity=3.141592653589793
- joint wrist_2_joint: limit lower=-6.283185307179586 upper=6.283185307179586 effort=28.0 velocity=3.141592653589793 -> lower=-3.141593 upper=3.141593 effort=28.0 velocity=3.141592653589793
- joint wrist_3_joint: limit lower=-6.283185307179586 upper=6.283185307179586 effort=28.0 velocity=3.141592653589793 -> lower=-3.141593 upper=3.141593 effort=28.0 velocity=3.141592653589793
