Commit message: Reorganise the robot assets by device, and drop the bare UR5e
The vendored description was laid out by upstream ROS package, so one
package held the FT 300, the Wrist Camera and the D435i bracket, and the
D435i itself was split across three folders. It is now one folder per
device under assets/robot/ur5_robotiq/meshes/ (ur5, ft300, wrist_camera,
robotiq_2f85, d435i), each with visual/ and collision/, and every mesh
path in the URDF is relative to the URDF. The raw xacro output and the
xacro move to source/.

Mesh files are byte-identical; build_ur5_robotiq_urdf.py maps each
upstream package:// path through MESH_DIRS and stops on one it does not
cover. The regenerated URDF differs from the old one only in filename=
attributes, and the regenerated bracket hull is byte-identical.

Removed: the UR5e option (its URDF, meshes and configs/ur5e.yml, whose
cspace weights are now TUNED_CSPACE in the config builder), the
ur5e-only clip_joint_limits.py and convert_v1_robot_yaml.py, the
duplicate bracket collision mesh and the unused ur_to_robotiq_adapter.
configs/ur5_robotiq.yml keeps its spheres; only its two paths become
repo-relative. Rebuilding it refits the spheres non-deterministically,
and a rerun missed the builder's own coverage bar, so it was not rebuilt.

check_robot_cfg.py could not load ur5_robotiq at all (paths hard-coded
to ur_description) and, once it could, planned with the base's
mask-only spheres inside the table. It now reads rig.ROBOTS and drops
SEGMENTER_ONLY like planner_server does; plan_pose succeeds.

Verified in Isaac Sim: baseline 59 plans, 0 failures, 0 voxels;
pick_place 32 plans, 0 failures, block shuttling between
[0.450, +/-0.400].

Co-Authored-By: Claude Opus 5.5 <noreply@anthropic.com>

File: assets/robot/ur5_robotiq/source/ur5_robotiq.raw.urdf (robot description, URDF)
Before this commit: robot ur5_robotiq, 44 links, 43 joints
Links:
- link realsense_link: geometry collision box size=0.02505 0.09 0.025; visual mesh filename=package://realsense2_description/meshes/d435.dae

File: assets/robot/ur5_robotiq/source/ur5_robotiq.urdf.xacro (robot description, xacro)
@@ -4,5 +4,9 @@
      only thing removed is the MiR100 chassis, so the arm stands on the ground
      instead of on the mobile base. Mounting transforms are copied verbatim
-     from mir_description/urdf/include/mir_100_v1.urdf.xacro. -->
+     from mir_description/urdf/include/mir_100_v1.urdf.xacro.
+     Kept as the record of how source/ur5_robotiq.raw.urdf was produced, not
+     as something to run: the include paths below point at a scratch checkout
+     of the upstream packages that no longer exists. To regenerate, clone
+     mir_ur5_humble's dependencies and point them there. -->
 <robot xmlns:xacro="http://ros.org/wiki/xacro" name="ur5_robotiq">
   <xacro:include filename="/tmp/claude-1000/-media-eencku-2TBDATA-yusian-ubuntu-UR5-curobo/7641c2f1-5308-4508-b802-402af3a1f5bb/scratchpad/mir_ur5/mir_robot/mir_description/urdf/include/common_properties.urdf.xacro"/>

File: assets/robot/ur5_robotiq/ur5_robotiq.urdf (robot description, URDF)
Before this commit: robot ur5_robotiq, 46 links, 45 joints
Links:
- link base_link_inertia: geometry collision mesh filename=meshes/ur5/collision/base.stl; visual mesh filename=meshes/ur5/visual/base.dae
- link camera_mount: geometry collision mesh filename=meshes/d435i/collision/bracket_hull.stl; visual mesh filename=meshes/d435i/visual/bracket.stl scale=0.001 0.001 0.001
- link forearm_link: geometry collision mesh filename=meshes/ur5/collision/forearm.stl; visual mesh filename=meshes/ur5/visual/forearm.dae
- link realsense_link: geometry collision box size=0.02505 0.09 0.025; visual mesh filename=meshes/d435i/visual/d435.dae
- link robotiq_85_base_link: geometry collision mesh filename=meshes/robotiq_2f85/collision/robotiq_base.stl; visual mesh filename=meshes/robotiq_2f85/visual/robotiq_base.dae
- link robotiq_85_left_finger_link: geometry collision mesh filename=meshes/robotiq_2f85/collision/left_finger.stl; visual mesh filename=meshes/robotiq_2f85/visual/left_finger.dae
- link robotiq_85_left_finger_tip_link: geometry collision mesh filename=meshes/robotiq_2f85/collision/left_finger_tip.stl; visual mesh filename=meshes/robotiq_2f85/visual/left_finger_tip.dae
- link robotiq_85_left_inner_knuckle_link: geometry collision mesh filename=meshes/robotiq_2f85/collision/left_inner_knuckle.stl; visual mesh filename=meshes/robotiq_2f85/visual/left_inner_knuckle.dae
- link robotiq_85_left_knuckle_link: geometry collision mesh filename=meshes/robotiq_2f85/collision/left_knuckle.stl; visual mesh filename=meshes/robotiq_2f85/visual/left_knuckle.dae
- link robotiq_85_right_finger_link: geometry collision mesh filename=meshes/robotiq_2f85/collision/right_finger.stl; visual mesh filename=meshes/robotiq_2f85/visual/right_finger.dae
- link robotiq_85_right_finger_tip_link: geometry collision mesh filename=meshes/robotiq_2f85/collision/right_finger_tip.stl; visual mesh filename=meshes/robotiq_2f85/visual/right_finger_tip.dae
- link robotiq_85_right_inner_knuckle_link: geometry collision mesh filename=meshes/robotiq_2f85/collision/right_inner_knuckle.stl; visual mesh filename=meshes/robotiq_2f85/visual/right_inner_knuckle.dae
- link robotiq_85_right_knuckle_link: geometry collision mesh filename=meshes/robotiq_2f85/collision/right_knuckle.stl; visual mesh filename=meshes/robotiq_2f85/visual/right_knuckle.dae
- link robotiq_ft300_mounting_plate: geometry collision cylinder length=0.013 radius=0.0375; visual mesh filename=meshes/ft300/visual/ft300_mounting_plate.stl
- link robotiq_ft300_sensor: geometry collision cylinder length=0.0348 radius=0.0375; visual mesh filename=meshes/ft300/visual/ft300.stl
- link robotiq_wrist_camera_link: geometry collision box size=0.045 0.020 0.0224; collision cylinder length=0.0135 radius=0.0375
- link shoulder_link: geometry collision mesh filename=meshes/ur5/collision/shoulder.stl; visual mesh filename=meshes/ur5/visual/shoulder.dae
- link upper_arm_link: geometry collision mesh filename=meshes/ur5/collision/upperarm.stl; visual mesh filename=meshes/ur5/visual/upperarm.dae
- link wrist_1_link: geometry collision mesh filename=meshes/ur5/collision/wrist1.stl; visual mesh filename=meshes/ur5/visual/wrist1.dae
- link wrist_2_link: geometry collision mesh filename=meshes/ur5/collision/wrist2.stl; visual mesh filename=meshes/ur5/visual/wrist2.dae
- link wrist_3_link: geometry collision mesh filename=meshes/ur5/collision/wrist3.stl; visual mesh filename=meshes/ur5/visual/wrist3.dae
