Commit message: Make the repo usable by someone else: install, check, license
README is rewritten to say in a few lines what the project does, with a
slot for the demo video, the headline numbers, and install steps that
follow the verified setup of this machine's environment: environment.yml
for Python 3.11, torch 2.7.0+cu128 and Isaac Sim 5.1, then cuRobo from
source on commit 8e734f3 with the [cu13] extra and packaging pinned back.

tools/check_pick_place.py is the regression check in one command: it
starts its own planner server, runs oracle episodes headless with mapping
off and on, and checks every pick holds, every place delivers, mapped
routes clear the slab and unmapped ones do not. ALL PASSED in 76 s here.

MIT license for the project; the vendored robot description keeps its
own. The Wrist Camera mesh is recorded as cleared for redistribution.

No more machine-specific paths: the run commands are relative, DISPLAY=:1
is gone, and the xacro's includes point at ROS package paths instead of
a scratch checkout that no longer exists.

HANDOVER.md is removed. What it knew that still applies was already in
the code next to each setting; the one thing that was not (update_world
taking effect a refresh late) moved into planner_server, and every
reference to it now says what it meant.

Co-Authored-By: Claude Opus 5.5 <noreply@anthropic.com>

File: assets/robot/ur5_robotiq/source/ur5_robotiq.urdf.xacro (robot description, xacro)
@@ -5,15 +5,16 @@
      instead of on the mobile base. Mounting transforms are copied verbatim
      from mir_description/urdf/include/mir_100_v1.urdf.xacro.
-     Kept as the record of how source/ur5_robotiq.raw.urdf was produced, not
-     as something to run: the include paths below point at a scratch checkout
-     of the upstream packages that no longer exists. To regenerate, clone
-     mir_ur5_humble's dependencies and point them there. -->
+     Kept as the record of how source/ur5_robotiq.raw.urdf was produced. The
+     includes resolve through ROS package paths, so it expands in a ROS 2
+     workspace that has mir_ur5_humble's packages built (mir_description,
+     ur_description, realsense2_description, robotiq_description):
+         xacro ur5_robotiq.urdf.xacro > ur5_robotiq.raw.urdf -->
 <robot xmlns:xacro="http://ros.org/wiki/xacro" name="ur5_robotiq">
-  <xacro:include filename="/tmp/claude-1000/-media-eencku-2TBDATA-yusian-ubuntu-UR5-curobo/7641c2f1-5308-4508-b802-402af3a1f5bb/scratchpad/mir_ur5/mir_robot/mir_description/urdf/include/common_properties.urdf.xacro"/>
-  <xacro:include filename="/tmp/claude-1000/-media-eencku-2TBDATA-yusian-ubuntu-UR5-curobo/7641c2f1-5308-4508-b802-402af3a1f5bb/scratchpad/mir_ur5/Universal_Robots_ROS2_Description/urdf/ur_macro.xacro"/>
-  <xacro:include filename="/tmp/claude-1000/-media-eencku-2TBDATA-yusian-ubuntu-UR5-curobo/7641c2f1-5308-4508-b802-402af3a1f5bb/scratchpad/mir_ur5/realsense2_description/urdf/_d435i.urdf.xacro"/>
-  <xacro:include filename="/tmp/claude-1000/-media-eencku-2TBDATA-yusian-ubuntu-UR5-curobo/7641c2f1-5308-4508-b802-402af3a1f5bb/scratchpad/mir_ur5/mir_robot/mir_description/urdf/include/robotiq_wrist_stack.xacro"/>
-  <xacro:include filename="/tmp/claude-1000/-media-eencku-2TBDATA-yusian-ubuntu-UR5-curobo/7641c2f1-5308-4508-b802-402af3a1f5bb/scratchpad/mir_ur5/mir_robot/mir_description/urdf/include/robotiq_gripper_macro.xacro"/>
-  <xacro:property name="ur_cfg" value="/tmp/claude-1000/-media-eencku-2TBDATA-yusian-ubuntu-UR5-curobo/7641c2f1-5308-4508-b802-402af3a1f5bb/scratchpad/mir_ur5/Universal_Robots_ROS2_Description/config/ur5"/>
+  <xacro:include filename="$(find mir_description)/urdf/include/common_properties.urdf.xacro"/>
+  <xacro:include filename="$(find ur_description)/urdf/ur_macro.xacro"/>
+  <xacro:include filename="$(find realsense2_description)/urdf/_d435i.urdf.xacro"/>
+  <xacro:include filename="$(find mir_description)/urdf/include/robotiq_wrist_stack.xacro"/>
+  <xacro:include filename="$(find mir_description)/urdf/include/robotiq_gripper_macro.xacro"/>
+  <xacro:property name="ur_cfg" value="$(find ur_description)/config/ur5"/>
   <!-- The arm stands on the floor; no chassis, no cabinet. -->
   <link name="world"/>
